File: hardware/kicad/link/vgacorne-link.kicad_sch (KiCad schematic)
At the start: 5 parts, among them J1 DE-15F (VGA), J2 JST-SH pigtail

Commit message: Use the Amphenol FCI 10090929-S154XLF VGA socket
A vertical HD-15 socket with 4-40 clinch nuts and board locks, in stock
at Digi-Key. The board locks, soldered into the plated mounting holes,
tie the shell (and through the jackscrews, the case) to GND. The library
gains a copy of KiCad's vertical HD-15 footprint with the 1.2 mm pin
holes and 3.1 mm board-lock holes Amphenol specifies.

Keystone 7229 jackscrews (0.187" hex, 0.25" stud) fix it to the 1.6 mm
wall; the docs cover soldering the board locks, clipping the pin tails
and checking the board-to-flange height on the first part.

Co-Authored-By: Claude Opus 5.5 (1M context) <noreply@anthropic.com>
Parts:
- J1: value DE-15F (VGA) -> 10090929-S154XLF; footprint Connector_Dsub:DSUB-15-HD_Socket_Vertical_P2.29x1.98mm_MountingHoles -> vgacorne:DSUB-15-HD_Socket_Vertical_P2.29x1.98mm_Amphenol_10090929; MPN (none) -> Amphenol FCI 10090929-S154XLF
Changed lines of the file:
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@@
 			)
 		)
-		(property "Value" "DE-15F (VGA)"
+		(property "Value" "10090929-S154XLF"
 			(at 36.83 57.15 0)
 			(effects
@@
 			)
 		)
-		(property "Footprint" "Connector_Dsub:DSUB-15-HD_Socket_Vertical_P2.29x1.98mm_MountingHoles"
+		(property "Footprint" "vgacorne:DSUB-15-HD_Socket_Vertical_P2.29x1.98mm_Amphenol_10090929"
 			(at 44.45 76.2 0)
 			(effects
@@
 			)
 		)
-		(property "Description" "HD-15 female, vertical PCB mount, 4-40 threaded inserts"
+		(property "Description" "HD-15 female, vertical PCB mount, 4-40 clinch nuts with board locks: solder the locks, they ground the shell and, through the jackscrews, the case"
 			(at 44.45 76.2 0)
 			(effects
+				(font (size 1.27 1.27))
+				(hide yes)
+			)
+		)
+		(property "MPN" "Amphenol FCI 10090929-S154XLF"
+			(at 44.45 76.2 0)
+			(effects

Commit message: Route the VGA daughterboard with Freerouting
hardware/route.py drives Freerouting directly (the KiCad MCP's autorouter
trips over a pcbnew/Python 3.14 binding bug): signals first with the
ground pours as planes, then ground as tracks round the locked signals,
then the pours and ground stitching vias. The daughterboard routes
completely and passes DRC.

To make it routable:
- the 10-pin link order now follows the DE-15 under the pigtail pads
  (J3 on both halves follows; the pigtail stays 1:1, +5 V on pin 1);
- the pigtail pads are shorter and at the board edge, leaving a via
  channel above the connector;
- the socket keeps KiCad's 1.6 mm pads round Amphenol's 1.2 mm holes,
  so a track fits between pins;
- both cable-variant jumpers sit together by pins 9 and 15.

generate.py --force pcbs now leaves boards with tracks alone.

Co-Authored-By: Claude Opus 5.5 (1M context) <noreply@anthropic.com>
Connections:
- net GND: now also J2.10 (Pin_10), J2.9 (Pin_9); no longer J2.2 (Pin_2), J2.7 (Pin_7)
- net LINK_B: now also J2.7 (Pin_7); no longer J2.9 (Pin_9)
- net LINK_C: now also J2.6 (Pin_6); no longer J2.10 (Pin_10)
- net LINK_DET: now also J2.2 (Pin_2); no longer J2.6 (Pin_6)
- net LINK_S0: now also J2.4 (Pin_4); no longer J2.3 (Pin_3)
- net LINK_S1: now also J2.3 (Pin_3); no longer J2.4 (Pin_4)
Changed lines of the file:
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@@
-	(wire
-		(pts
-			(xy 90.17 59.69)
-			(xy 87.63 59.69)
-		)
-		(stroke
-			(width 0)
-			(type default)
-		)
-	)
-	(label "+5V_LINK"
-		(at 87.63 59.69 180)
-		(fields_autoplaced yes)
-		(effects
-			(font (size 1.27 1.27))
-			(justify right bottom)
-		)
-	)
-	(wire
-		(pts
-			(xy 90.17 64.77)
-			(xy 87.63 64.77)
-		)
-		(stroke
-			(width 0)
-			(type default)
-		)
-	)
-	(label "LINK_S0"
-		(at 87.63 64.77 180)
-		(fields_autoplaced yes)
-		(effects
-			(font (size 1.27 1.27))
-			(justify right bottom)
-		)
-	)
-	(wire
-		(pts
-			(xy 90.17 67.31)
-			(xy 87.63 67.31)
-		)
-		(stroke
-			(width 0)
-			(type default)
-		)
-	)
-	(label "LINK_S1"
-		(at 87.63 67.31 180)
-		(fields_autoplaced yes)
-		(effects
-			(font (size 1.27 1.27))
-			(justify right bottom)
-		)
-	)
-	(wire
-		(pts
-			(xy 90.17 69.85)
-			(xy 87.63 69.85)
-		)
-		(stroke
-			(width 0)
-			(type default)
-		)
-	)
-	(label "LINK_S2"
-		(at 87.63 69.85 180)
-		(fields_autoplaced yes)
-		(effects
-			(font (size 1.27 1.27))
-			(justify right bottom)
-		)
-	)
-	(wire
-		(pts
-			(xy 90.17 72.39)
-			(xy 87.63 72.39)
-		)
-		(stroke
-			(width 0)
-			(type default)
-		)
-	)
-	(label "LINK_DET"
-		(at 87.63 72.39 180)
-		(fields_autoplaced yes)
-		(effects
-			(font (size 1.27 1.27))
-			(justify right bottom)
-		)
-	)
-	(wire
-		(pts
-			(xy 90.17 77.47)
-			(xy 87.63 77.47)
-		)
-		(stroke
-			(width 0)
-			(type default)
-		)
-	)
-	(label "LINK_A"
-		(at 87.63 77.47 180)
-		(fields_autoplaced yes)
-		(effects
-			(font (size 1.27 1.27))
-			(justify right bottom)
-		)
-	)
 	(wire
 		(pts
@@
 		)
 	)
-	(label "LINK_B"
-		(at 87.63 80.01 180)
-		(fields_autoplaced yes)
-		(effects
-			(font (size 1.27 1.27))
-			(justify right bottom)
-		)
-	)
 	(wire
 		(pts
@@
 		)
 	)
-	(label "LINK_C"
-		(at 87.63 82.55 180)
-		(fields_autoplaced yes)
-		(effects
-			(font (size 1.27 1.27))
-			(justify right bottom)
-		)
-	)
-	(wire
-		(pts
-			(xy 90.17 62.23)
-			(xy 87.63 62.23)
+	(wire
+		(pts
+			(xy 87.63 80.01)
+			(xy 87.63 82.55)
+		)
+		(stroke
+			(width 0)
+			(type default)
+		)
+	)
+	(junction
+		(at 87.63 80.01)
+		(diameter 0)
+		(color 0 0 0 0)
+	)
+	(wire
+		(pts
+			(xy 87.63 80.01)
+			(xy 85.09 80.01)
 		)
 		(stroke
@@
 	(symbol
 		(lib_id "power:GND")
-		(at 87.63 62.23 270)
+		(at 85.09 80.01 270)
 		(unit 1)
 		(exclude_from_sim no)
@@
 		(dnp no)
 		(property "Reference" "#PWR006"
-			(at 88.9 62.23 0)
+			(at 86.36 80.01 0)
 			(effects
 				(font (size 1.27 1.27))
@@
 		)
 		(property "Value" "GND"
-			(at 88.9 64.77 0)
+			(at 86.36 82.55 0)
 			(effects
 				(font (size 1.27 1.27))
@@
 		)
 		(property "Footprint" ""
-			(at 87.63 62.23 0)
+			(at 85.09 80.01 0)
 			(effects
 				(font (size 1.27 1.27))
@@
 		)
 		(property "Datasheet" ""
-			(at 87.63 62.23 0)
+			(at 85.09 80.01 0)
 			(effects
 				(font (size 1.27 1.27))
@@
 		)
 		(property "Description" "Power symbol creates a global label with name \"GND\" , ground"
-			(at 87.63 62.23 0)
+			(at 85.09 80.01 0)
 			(effects
 				(font (size 1.27 1.27))
@@
 	(wire
 		(pts
+			(xy 90.17 59.69)
+			(xy 87.63 59.69)
+		)
+		(stroke
+			(width 0)
+			(type default)
+		)
+	)
+	(label "+5V_LINK"
+		(at 87.63 59.69 180)
+		(fields_autoplaced yes)
+		(effects
+			(font (size 1.27 1.27))
+			(justify right bottom)
+		)
+	)
+	(wire
+		(pts
+			(xy 90.17 62.23)
+			(xy 87.63 62.23)
+		)
+		(stroke
+			(width 0)
+			(type default)
+		)
+	)
+	(label "LINK_DET"
+		(at 87.63 62.23 180)
+		(fields_autoplaced yes)
+		(effects
+			(font (size 1.27 1.27))
+			(justify right bottom)
+		)
+	)
+	(wire
+		(pts
+			(xy 90.17 64.77)
+			(xy 87.63 64.77)
+		)
+		(stroke
+			(width 0)
+			(type default)
+		)
+	)
+	(label "LINK_S1"
+		(at 87.63 64.77 180)
+		(fields_autoplaced yes)
+		(effects
+			(font (size 1.27 1.27))
+			(justify right bottom)
+		)
+	)
+	(wire
+		(pts
+			(xy 90.17 67.31)
+			(xy 87.63 67.31)
+		)
+		(stroke
+			(width 0)
+			(type default)
+		)
+	)
+	(label "LINK_S0"
+		(at 87.63 67.31 180)
+		(fields_autoplaced yes)
+		(effects
+			(font (size 1.27 1.27))
+			(justify right bottom)
+		)
+	)
+	(wire
+		(pts
+			(xy 90.17 69.85)
+			(xy 87.63 69.85)
+		)
+		(stroke
+			(width 0)
+			(type default)
+		)
+	)
+	(label "LINK_S2"
+		(at 87.63 69.85 180)
+		(fields_autoplaced yes)
+		(effects
+			(font (size 1.27 1.27))
+			(justify right bottom)
+		)
+	)
+	(wire
+		(pts
+			(xy 90.17 72.39)
+			(xy 87.63 72.39)
+		)
+		(stroke
+			(width 0)
+			(type default)
+		)
+	)
+	(label "LINK_C"
+		(at 87.63 72.39 180)
+		(fields_autoplaced yes)
+		(effects
+			(font (size 1.27 1.27))
+			(justify right bottom)
+		)
+	)
+	(wire
+		(pts
 			(xy 90.17 74.93)
 			(xy 87.63 74.93)
@@
 		)
 	)
-	(symbol
-		(lib_id "power:GND")
-		(at 87.63 74.93 270)
-		(unit 1)
-		(exclude_from_sim no)
-		(in_bom no)
-		(on_board no)
-		(dnp no)
-		(property "Reference" "#PWR007"
-			(at 88.9 74.93 0)
-			(effects
-				(font (size 1.27 1.27))
-				(justify left)
-				(hide yes)
-			)
-		)
-		(property "Value" "GND"
-			(at 88.9 77.47 0)
-			(effects
-				(font (size 1.27 1.27))
-				(justify left)
-			)
-		)
-		(property "Footprint" ""
-			(at 87.63 74.93 0)
-			(effects
-				(font (size 1.27 1.27))
-				(hide yes)
-			)
-		)
-		(property "Datasheet" ""
-			(at 87.63 74.93 0)
-			(effects
-				(font (size 1.27 1.27))
-				(hide yes)
-			)
-		)
-		(property "Description" "Power symbol creates a global label with name \"GND\" , ground"
-			(at 87.63 74.93 0)
-			(effects
-				(font (size 1.27 1.27))
-				(hide yes)
-			)
-		)
-		(pin "1"
-		)
-		(instances
-			(project "vgacorne-link"
-				(path "/6c8c1982-d650-5c52-8c9c-77d9b895e034"
-					(reference "#PWR007")
-					(unit 1)
-				)
-			)
+	(label "LINK_B"
+		(at 87.63 74.93 180)
+		(fields_autoplaced yes)
+		(effects
+			(font (size 1.27 1.27))
+			(justify right bottom)
+		)
+	)
+	(wire
+		(pts
+			(xy 90.17 77.47)
+			(xy 87.63 77.47)
+		)
+		(stroke
+			(width 0)
+			(type default)
+		)
+	)
+	(label "LINK_A"
+		(at 87.63 77.47 180)
+		(fields_autoplaced yes)
+		(effects
+			(font (size 1.27 1.27))
+			(justify right bottom)
 		)
 	)
@@
 		(on_board no)
 		(dnp no)
-		(property "Reference" "#PWR008"
+		(property "Reference" "#PWR007"
 			(at 125.73 181.61 0)
 			(effects
@@
 			(project "vgacorne-link"
 				(path "/6c8c1982-d650-5c52-8c9c-77d9b895e034"
-					(reference "#PWR008")
+					(reference "#PWR007")
 					(unit 1)
 				)
@@
 		(on_board no)
 		(dnp no)
-		(property "Reference" "#PWR009"
+		(property "Reference" "#PWR008"
 			(at 27.94 29.21 0)
 			(effects
@@
 			(project "vgacorne-link"
 				(path "/6c8c1982-d650-5c52-8c9c-77d9b895e034"
-					(reference "#PWR009")
+					(reference "#PWR008")
 					(unit 1)
 				)
