File: hardware/kicad/satellite/vgacorne-satellite.kicad_sch (KiCad schematic)
At the start: 110 parts, among them J3 SM10B-SRSS-TB, SW1 C0R0, SW10 C3R0, SW11 C3R1, SW12 C3R2, SW13 C4R0, SW14 C4R1, SW15 C4R2, SW16 C5R0, SW17 C5R1, SW18 C5R2, SW19 T0, SW2 C0R1, SW20 T1, SW21 T2, SW3 C0R2, SW4 C1R0, SW5 C1R1, SW6 C1R2, SW7 C2R0, SW8 C2R1, SW9 C2R2, U11 SN74LV4051APWR, U12 SN74LV4051APWR, U13 SN74LV4051APWR, U2 TLV75733PDBVR, U5 TLV9064IPWR, U6 SRV05-4, U7 SRV05-4

Commit message: Add trackpad, mouse column and scroll wheel; move MCU and ports
Layout
- MCU module, USB-C and trackpad move to the right half; the left half
  is now the passive satellite.
- VGA daughterboard bay moves to the inner-back corner so both cables
  leave from the back face. The bay sits 4.5 mm further back than the
  keys need, so both halves are 116 mm deep.
- Azoteq TPS65 trackpad, landscape, right beside Y/H/N under a 1 mm
  overlay. The MCU module moves to a PCB ear behind it, next to the
  VGA bay. trackpad.py selects the pad (TPS65 or 40 mm Cirque); the
  case pocket, J5 connector and QMK driver follow the selection.
- Left half: a mouse column beside T/G/B with a scroll wheel (Bourns
  PEC12R) at the top and left/right-click HE keys beside G and B.

Circuits and firmware
- Mux channels reassigned so the satellite's mouse keys and wheel fill
  its three spare channels. The wheel's A/B contacts are summed into
  four voltage levels on one channel.
- QMK: 44-key LAYOUT and a wheel decoder that feeds QMK's quadrature
  encoder driver. Trackpad on I2C1, with rules.mk now generated. The
  host test covers the wheel.
- libhmk: MS_BTN1/MS_BTN2 on the mouse keys (no encoder support).

Case and renders
- Smoother milled case: 7.25 mm walls, 25 mm minimum outside radius
  and a flat back face at the ports.
- render.py builds Blender Cycles renders from the design geometry.

Co-Authored-By: Claude Opus 5.5 (1M context) <noreply@anthropic.com>
Parts:
- added C122, C123: 100n, Capacitor_SMD:C_0402_1005Metric, symbol Device:C
- added C222, C223: 4.7n, Capacitor_SMD:C_0402_1005Metric, symbol Device:C
- added C5: 1n, Capacitor_SMD:C_0402_1005Metric, symbol Device:C
- added ENC1: PEC12R-2217F-N0024, Rotary_Encoder:RotaryEncoder_Bourns_Horizontal_PEC12R-2x17F-Nxxxx, symbol Device:RotaryEncoder
- added H8: M2 standoff, vgacorne:Standoff_M2, symbol Mechanical:MountingHole
- added HE22, HE23: DRV5055A3QDBZR, Package_TO_SOT_SMD:SOT-23, symbol Sensor_Magnetic:DRV5055A3xDBZxQ1
- added R21, R22: 10k, Resistor_SMD:R_0402_1005Metric, symbol Device:R
- added R23: 47k, Resistor_SMD:R_0402_1005Metric, symbol Device:R
- added R24: 100k, Resistor_SMD:R_0402_1005Metric, symbol Device:R
- added SW22: M0, vgacorne:SW_HE_MX_1u, symbol Mechanical:MountingHole
- added SW23: M1, vgacorne:SW_HE_MX_1u, symbol Mechanical:MountingHole
Connections:
- net +3.3VA: now also C122.1, C123.1, HE22.1 (VCC), HE23.1 (VCC), R21.2, R22.2
- net GND: now also C122.2, C123.2, C222.2, C223.2, C5.2, ENC1.C, HE22.3 (GND), HE23.3 (GND); no longer U11.2 (A6), U11.4 (A7), U12.4 (A7)
- net HE_C2R0: now also U11.2 (A6); no longer U12.13 (A0)
- net HE_C2R1: now also U11.4 (A7); no longer U12.14 (A1)
- net HE_C2R2: now also U12.13 (A0); no longer U12.15 (A2)
- net HE_C3R0: now also U12.14 (A1); no longer U12.12 (A3)
- net HE_C3R1: now also U12.15 (A2); no longer U12.1 (A4)
- net HE_C3R2: now also U12.12 (A3); no longer U12.5 (A5)
- net HE_C4R0: now also U12.1 (A4); no longer U13.13 (A0)
- net HE_C4R1: now also U12.5 (A5); no longer U13.14 (A1)
- net HE_C4R2: now also U12.2 (A6); no longer U13.15 (A2)
- net HE_C5R0: now also U13.13 (A0); no longer U13.12 (A3)
- net HE_C5R1: now also U13.14 (A1); no longer U13.1 (A4)
- net HE_C5R2: now also U13.15 (A2); no longer U13.5 (A5)
- net HE_T0: now also U12.4 (A7); no longer U12.2 (A6)
- net HE_T1: now also U13.12 (A3); no longer U13.2 (A6)
- net HE_T2: now also U13.1 (A4); no longer U13.4 (A7)
- new net HE_M0: C222.1, HE22.2 (OUT), U13.5 (A5)
- new net HE_M1: C223.1, HE23.2 (OUT), U13.2 (A6)
- new net WHEEL: C5.1, R23.2, R24.2, U13.4 (A7)
- new net WHEEL_A: ENC1.A, R21.1, R23.1
- new net WHEEL_B: ENC1.B, R22.1, R24.1
Other:
- note added: "Scroll wheel: A/B summed into one level on mux C channel 7"
- title: VGACorne - satellite (right) half -> VGACorne - satellite (left) half

Commit message: Replace the scroll wheel with a rotary encoder knob
The left half's mouse column now runs, top to bottom: right click beside
T, left click beside G, and a rotary encoder with a knob beside B, all
in line with column 5's rows.
- Encoder: Bourns PEC12R-4220F-N0024 (upright, 20 mm shaft, 24
  detents, no switch). It sits in a normal 14 mm plate cutout, which
  replaces the wheel notch. The knob is 16 mm across.
- Same readout as before: the A/B contacts are summed into four levels
  on the satellite's last spare mux channel. Nets, QMK defines and code
  are renamed from wheel to encoder (ENC, HE_ENCODER_*).
- The link connector J3 goes back to its original spot, now that the
  encoder legs are elsewhere.
- Docs, BOM, PCB images and renders regenerated.

Co-Authored-By: Claude Opus 5.5 (1M context) <noreply@anthropic.com>
Parts:
- ENC1: value PEC12R-2217F-N0024 -> PEC12R-4220F-N0024; footprint Rotary_Encoder:RotaryEncoder_Bourns_Horizontal_PEC12R-2x17F-Nxxxx -> Rotary_Encoder:RotaryEncoder_Bourns_Vertical_PEC12R-3x17F-Nxxxx; MPN PEC12R-2217F-N0024 -> PEC12R-4220F-N0024
Connections:
- net WHEEL renamed ENC
- net WHEEL_A renamed ENC_A
- net WHEEL_B renamed ENC_B
Other:
- note added: "Rotary encoder: A/B summed into one level on mux C channel 7"
- note removed: "Scroll wheel: A/B summed into one level on mux C channel 7"
Changed lines of the file:
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@@
 		)
 	)
-	(text "Scroll wheel: A/B summed into one level on mux C channel 7"
+	(text "Rotary encoder: A/B summed into one level on mux C channel 7"
 		(exclude_from_sim no)
 		(at 292.1 132.54 0)
@@
 			)
 		)
-		(property "Description" "8:1 analog mux C (C5R0, C5R1, C5R2, T1, T2, M0, M1, WHEEL)"
+		(property "Description" "8:1 analog mux C (C5R0, C5R1, C5R2, T1, T2, M0, M1, ENC)"
 			(at 154.94 238.76 0)
 			(effects
@@
 		)
 	)
-	(label "WHEEL"
+	(label "ENC"
 		(at 167.64 248.92 0)
 		(fields_autoplaced yes)
@@
 			)
 		)
-		(property "Value" "PEC12R-2217F-N0024"
+		(property "Value" "PEC12R-4220F-N0024"
 			(at 322.58 153.67 0)
 			(effects
@@
 			)
 		)
-		(property "Footprint" "Rotary_Encoder:RotaryEncoder_Bourns_Horizontal_PEC12R-2x17F-Nxxxx"
+		(property "Footprint" "Rotary_Encoder:RotaryEncoder_Bourns_Vertical_PEC12R-3x17F-Nxxxx"
 			(at 316.23 154.94 0)
 			(effects
@@
 			)
 		)
-		(property "Description" "Scroll wheel: 24 detents, shaft 10 mm above the PCB; 18 x 6 mm rubber wheel on the shaft, which is cut to 13 mm"
+		(property "Description" "Rotary encoder with a knob: 24 detents, 20 mm shaft, no bushing, no switch (same PCB layout as the -3 bushing version)"
 			(at 316.23 154.94 0)
 			(effects
@@
 			)
 		)
-		(property "MPN" "PEC12R-2217F-N0024"
+		(property "MPN" "PEC12R-4220F-N0024"
 			(at 316.23 154.94 0)
 			(effects
@@
 		)
 	)
-	(label "WHEEL_A"
+	(label "ENC_A"
 		(at 306.07 152.4 180)
 		(fields_autoplaced yes)
@@
 		)
 	)
-	(label "WHEEL_B"
+	(label "ENC_B"
 		(at 306.07 157.48 180)
 		(fields_autoplaced yes)
@@
 		)
 	)
-	(label "WHEEL_A"
+	(label "ENC_A"
 		(at 349.25 147.32 90)
 		(fields_autoplaced yes)
@@
 		)
 	)
-	(label "WHEEL_B"
+	(label "ENC_B"
 		(at 367.03 147.32 90)
 		(fields_autoplaced yes)
@@
 		)
 	)
-	(label "WHEEL_A"
+	(label "ENC_A"
 		(at 384.81 147.32 90)
 		(fields_autoplaced yes)
@@
 		)
 	)
-	(label "WHEEL"
+	(label "ENC"
 		(at 384.81 160.02 270)
 		(fields_autoplaced yes)
@@
 		)
 	)
-	(label "WHEEL_B"
+	(label "ENC_B"
 		(at 403.86 147.32 90)
 		(fields_autoplaced yes)
@@
 		)
 	)
-	(label "WHEEL"
+	(label "ENC"
 		(at 403.86 160.02 270)
 		(fields_autoplaced yes)
@@
 		)
 	)
-	(label "WHEEL"
+	(label "ENC"
 		(at 422.91 147.32 90)
 		(fields_autoplaced yes)

Commit message: Fix design audit findings
Electrical:
- Re-map the castellated module's pads so neighbours on each edge follow
  the LQFP: USB D+/D- together between grounds at the corner nearest the
  USB-C, the six ADC inputs grouped beside +3.3VA, a ground away from the
  select lines.
- Put 1k between each DRV5055 output and its 4.7n cap (TI: no capacitor
  straight on the output).
- STM32F446 module: pull PB2/BOOT1 down so BOOT reaches DFU; pull PA10 up.
- Replace the XC6206 with a second TLV75733, and the link polyfuse with a
  TPS2051C switch (soft start, current limit) so hot-plugging the satellite
  can't brown out the MCU. F1 is now 750 mA.
- USB net class 0.4/0.15 mm: ~97 ohm differential against the pour on both
  2-layer boards (was ~120).
- BOM gains a Tolerance column; part numbers for the F446 crystal.

Mechanical:
- Case foam 2 mm, leaving 0.5 mm under the bottom-side parts (the old stack
  pressed the foam into every sensor).
- USB-C overhangs the ear by 0.46 mm and the opening takes a spec-maximum
  overmould (13.95 x 8.1 mm); the old 11 x 6 mm stopped most plugs short.
- DE-15 rear-mount cutout 20.5 x 11.4 mm; floor pockets under the USB-C and
  encoder pins; plate foam clears the module and the encoder's pins.
- Knob 11.5 mm tall so it clears the encoder's collar.

Docs, PCB images and renders updated to match.

Co-Authored-By: Claude Opus 5.5 (1M context) <noreply@anthropic.com>
Parts:
- added R301, R302, R303, R304, R305, R306, R307, R308, R309, R310, R311, R312, R313, R314, R315, R316, R317, R318, R319, R320, R321, R322, R323: 1k, Resistor_SMD:R_0402_1005Metric, symbol Device:R
Connections:
- net HE_C0R0: now also R301.2; no longer HE1.2 (OUT)
- net HE_C0R1: now also R302.2; no longer HE2.2 (OUT)
- net HE_C0R2: now also R303.2; no longer HE3.2 (OUT)
- net HE_C1R0: now also R304.2; no longer HE4.2 (OUT)
- net HE_C1R1: now also R305.2; no longer HE5.2 (OUT)
- net HE_C1R2: now also R306.2; no longer HE6.2 (OUT)
- net HE_C2R0: now also R307.2; no longer HE7.2 (OUT)
- net HE_C2R1: now also R308.2; no longer HE8.2 (OUT)
- net HE_C2R2: now also R309.2; no longer HE9.2 (OUT)
- net HE_C3R0: now also R310.2; no longer HE10.2 (OUT)
- net HE_C3R1: now also R311.2; no longer HE11.2 (OUT)
- net HE_C3R2: now also R312.2; no longer HE12.2 (OUT)
- net HE_C4R0: now also R313.2; no longer HE13.2 (OUT)
- net HE_C4R1: now also R314.2; no longer HE14.2 (OUT)
- net HE_C4R2: now also R315.2; no longer HE15.2 (OUT)
- net HE_C5R0: now also R316.2; no longer HE16.2 (OUT)
- net HE_C5R1: now also R317.2; no longer HE17.2 (OUT)
- net HE_C5R2: now also R318.2; no longer HE18.2 (OUT)
- net HE_M0: now also R322.2; no longer HE22.2 (OUT)
- net HE_M1: now also R323.2; no longer HE23.2 (OUT)
- net HE_T0: now also R319.2; no longer HE19.2 (OUT)
- net HE_T1: now also R320.2; no longer HE20.2 (OUT)
- net HE_T2: now also R321.2; no longer HE21.2 (OUT)
- new net HE_C0R0_OUT: HE1.2 (OUT), R301.1
- new net HE_C0R1_OUT: HE2.2 (OUT), R302.1
- new net HE_C0R2_OUT: HE3.2 (OUT), R303.1
- new net HE_C1R0_OUT: HE4.2 (OUT), R304.1
- new net HE_C1R1_OUT: HE5.2 (OUT), R305.1
- new net HE_C1R2_OUT: HE6.2 (OUT), R306.1
- new net HE_C2R0_OUT: HE7.2 (OUT), R307.1
- new net HE_C2R1_OUT: HE8.2 (OUT), R308.1
- new net HE_C2R2_OUT: HE9.2 (OUT), R309.1
- new net HE_C3R0_OUT: HE10.2 (OUT), R310.1
- new net HE_C3R1_OUT: HE11.2 (OUT), R311.1
- new net HE_C3R2_OUT: HE12.2 (OUT), R312.1
- new net HE_C4R0_OUT: HE13.2 (OUT), R313.1
- new net HE_C4R1_OUT: HE14.2 (OUT), R314.1
- new net HE_C4R2_OUT: HE15.2 (OUT), R315.1
- new net HE_C5R0_OUT: HE16.2 (OUT), R316.1
- new net HE_C5R1_OUT: HE17.2 (OUT), R317.1
- new net HE_C5R2_OUT: HE18.2 (OUT), R318.1
- new net HE_M0_OUT: HE22.2 (OUT), R322.1
- new net HE_M1_OUT: HE23.2 (OUT), R323.1
- new net HE_T0_OUT: HE19.2 (OUT), R319.1
- new net HE_T1_OUT: HE20.2 (OUT), R320.1
- new net HE_T2_OUT: HE21.2 (OUT), R321.1
Other:
- moved on the sheet: C102, C103, C104, C105, C106, C107, C108, C109, C110, C111, C112, C113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

Commit message: Route the VGA daughterboard with Freerouting
hardware/route.py drives Freerouting directly (the KiCad MCP's autorouter
trips over a pcbnew/Python 3.14 binding bug): signals first with the
ground pours as planes, then ground as tracks round the locked signals,
then the pours and ground stitching vias. The daughterboard routes
completely and passes DRC.

To make it routable:
- the 10-pin link order now follows the DE-15 under the pigtail pads
  (J3 on both halves follows; the pigtail stays 1:1, +5 V on pin 1);
- the pigtail pads are shorter and at the board edge, leaving a via
  channel above the connector;
- the socket keeps KiCad's 1.6 mm pads round Amphenol's 1.2 mm holes,
  so a track fits between pins;
- both cable-variant jumpers sit together by pins 9 and 15.

generate.py --force pcbs now leaves boards with tracks alone.

Co-Authored-By: Claude Opus 5.5 (1M context) <noreply@anthropic.com>
Connections:
- net GND: now also J3.10 (Pin_10), J3.9 (Pin_9); no longer J3.2 (Pin_2), J3.7 (Pin_7)
- net LINK_B: now also J3.7 (Pin_7); no longer J3.9 (Pin_9)
- net LINK_C: now also J3.6 (Pin_6); no longer J3.10 (Pin_10)
- net LINK_DET: now also J3.2 (Pin_2); no longer J3.6 (Pin_6)
- net LINK_S0: now also J3.4 (Pin_4); no longer J3.3 (Pin_3)
- net LINK_S1: now also J3.3 (Pin_3); no longer J3.4 (Pin_4)
